File: V67_cycletron/V67_cycletron.kicad_sch (KiCad schematic)
At the start: 41 parts, among them J1 USB_C_Receptacle_USB2.0_16P, J2 Screw_Terminal_01x02, J3 Screw_Terminal_01x14, J4 Screw_Terminal_01x02, U1 ESP32-S3-WROOM-1, U2 LM1117DT-3.3, U3 LM1117DT-5.0

Commit message: test commit, added schotsky diode
Parts:
- removed D1: 1N4001, Diode_THT:D_DO-41_SOD81_P10.16mm_Horizontal, symbol Diode:1N4001
- added D3: D_Schottky, Diode_SMD:D_SMA, symbol Device:D_Schottky
Connections:
- net +12V: now also U3.3 (VI), reg_5V_smoothing_caps_in1.1, D3.1 (K); no longer J2.1 (Pin_1)
- new net: D3.2 (A), J2.1 (Pin_1)
Changed lines of the file:
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@@
 	)
 	(junction
-		(at 29.21 63.5)
+		(at 88.9 71.12)
 		(diameter 0)
 		(color 0 0 0 0)
 	)
 	(junction
-		(at 88.9 71.12)
+		(at 170.18 87.63)
 		(diameter 0)
 		(color 0 0 0 0)
 	)
 	(junction
-		(at 170.18 87.63)
+		(at 29.21 63.5)
 		(diameter 0)
 		(color 0 0 0 0)
@@
 	)
 	(symbol
+		(lib_id "Device:D_Schottky")
+		(at 74.93 26.67 90)
+		(unit 1)
+		(exclude_from_sim no)
+		(in_bom yes)
+		(on_board yes)
+		(dnp no)
+		(fields_autoplaced yes)
+		(property "Reference" "D3"
+			(at 68.58 26.9875 0)
+			(effects
+				(font
+					(size 1.27 1.27)
+				)
+			)
+		)
+		(property "Value" "D_Schottky"
+			(at 71.12 26.9875 0)
+			(effects
+				(font
+					(size 1.27 1.27)
+				)
+			)
+		)
+		(property "Footprint" "Diode_SMD:D_SMA"
+			(at 74.93 26.67 0)
+			(effects
+				(font
+					(size 1.27 1.27)
+				)
+				(hide yes)
+			)
+		)
+		(property "Datasheet" "~"
+			(at 74.93 26.67 0)
+			(effects
+				(font
+					(size 1.27 1.27)
+				)
+				(hide yes)
+			)
+		)
+		(property "Description" "Schottky diode"
+			(at 74.93 26.67 0)
+			(effects
+				(font
+					(size 1.27 1.27)
+				)
+				(hide yes)
+			)
+		)
+		(pin "1"
+		)
+		(pin "2"
+		)
+		(instances
+			(project ""
+				(path "/490d8b32-3aea-4f11-93e7-a546853a1b13"
+					(reference "D3")
+					(unit 1)
+				)
+			)
+		)
+	)
+	(symbol
 		(lib_id "Device:C_Polarized")
 		(at 29.21 68.58 0)
@@
 	(symbol
 		(lib_id "power:+12V")
-		(at 21.59 63.5 90)
+		(at 29.21 63.5 90)
 		(unit 1)
 		(exclude_from_sim no)
@@
 		(fields_autoplaced yes)
 		(property "Reference" "#PWR01"
-			(at 25.4 63.5 0)
+			(at 33.02 63.5 0)
 			(effects
 				(font
@@
 		)
 		(property "Value" "+12V"
-			(at 17.78 63.5001 90)
+			(at 25.4 63.5001 90)
 			(effects
 				(font
@@
 		)
 		(property "Footprint" ""
-			(at 21.59 63.5 0)
+			(at 29.21 63.5 0)
 			(effects
 				(font
@@
 		)
 		(property "Datasheet" ""
-			(at 21.59 63.5 0)
+			(at 29.21 63.5 0)
 			(effects
 				(font
@@
 		)
 		(property "Description" "Power symbol creates a global label with name \"+12V\""
-			(at 21.59 63.5 0)
+			(at 29.21 63.5 0)
 			(effects
 				(font
@@
 	(symbol
 		(lib_id "power:+12V")
-		(at 74.93 22.86 180)
+		(at 74.93 30.48 180)
 		(unit 1)
 		(exclude_from_sim no)
@@
 		(fields_autoplaced yes)
 		(property "Reference" "#PWR033"
-			(at 74.93 19.05 0)
+			(at 74.93 26.67 0)
 			(effects
 				(font
@@
 		)
 		(property "Value" "+12V"
-			(at 74.93 27.94 0)
+			(at 74.9299 34.29 90)
 			(effects
 				(font
 					(size 1.27 1.27)
 				)
+				(justify left)
 			)
 		)
 		(property "Footprint" ""
-			(at 74.93 22.86 0)
+			(at 74.93 30.48 0)
 			(effects
 				(font
@@
 		)
 		(property "Datasheet" ""
-			(at 74.93 22.86 0)
+			(at 74.93 30.48 0)
 			(effects
 				(font
@@
 		)
 		(property "Description" "Power symbol creates a global label with name \"+12V\""
-			(at 74.93 22.86 0)
+			(at 74.93 30.48 0)
 			(effects
 				(font
@@
 					(unit 1)
 				)
-			)
-		)
-	)
-	(symbol
-		(lib_id "Diode:1N4001")
-		(at 25.4 63.5 180)
-		(unit 1)
-		(exclude_from_sim no)
-		(in_bom yes)
-		(on_board yes)
-		(dnp no)
-		(fields_autoplaced yes)
-		(property "Reference" "D1"
-			(at 25.4 57.15 0)
-			(effects
-				(font
-					(size 1.27 1.27)
-				)
-			)
-		)
-		(property "Value" "1N4001"
-			(at 25.4 59.69 0)
-			(effects
-				(font
-					(size 1.27 1.27)
-				)
-			)
-		)
-		(property "Footprint" "Diode_THT:D_DO-41_SOD81_P10.16mm_Horizontal"
-			(at 25.4 63.5 0)
-			(effects
-				(font
-					(size 1.27 1.27)
-				)
-				(hide yes)
-			)
-		)
-		(property "Datasheet" "http://www.vishay.com/docs/88503/1n4001.pdf"
-			(at 25.4 63.5 0)
-			(effects
-				(font
-					(size 1.27 1.27)
-				)
-				(hide yes)
-			)
-		)
-		(property "Description" "50V 1A General Purpose Rectifier Diode, DO-41"
-			(at 25.4 63.5 0)
-			(effects
-				(font
-					(size 1.27 1.27)
-				)
-				(hide yes)
-			)
-		)
-		(property "Sim.Device" "D"
-			(at 25.4 63.5 0)
-			(effects
-				(font
-					(size 1.27 1.27)
-				)
-				(hide yes)
-			)
-		)
-		(property "Sim.Pins" "1=K 2=A"
-			(at 25.4 63.5 0)
-			(effects
-				(font
-					(size 1.27 1.27)
-				)
-				(hide yes)
-			)
-		)
-		(pin "1"
-		)
-		(pin "2"
-		)
-		(instances
-			(project "V67_cycletron"
-				(path "/490d8b32-3aea-4f11-93e7-a546853a1b13"
-					(reference "D1")
-					(unit 1)
-				)

Commit message: got all parts to sync to jlcpcb
Parts:
- 3v3in1: renamed from reg_3v3_smoother_in1; footprint Capacitor_THT:CP_Radial_D6.3mm_P2.50mm -> Capacitor_SMD:CP_Elec_6.3x5.4; LCSC (none) -> C2749
- 3v3out1: renamed from reg_3v3_smoother_out1; footprint Capacitor_THT:CP_Radial_D5.0mm_P2.50mm -> Capacitor_SMD:CP_Elec_4x5.4; LCSC (none) -> C3343
- 5Vin1: renamed from reg_5V_smoothing_caps_in1; footprint Capacitor_THT:CP_Radial_D6.3mm_P2.50mm -> Capacitor_SMD:CP_Elec_6.3x5.4; LCSC (none) -> C2749
- 5Vout1: renamed from reg_5V_smoothing_caps_out1; footprint Capacitor_THT:CP_Radial_D5.0mm_P2.50mm -> Capacitor_SMD:CP_Elec_4x5.4; LCSC (none) -> C3343
- Boot1, En1: LCSC (none) -> C720477
- C1: renamed from C6; LCSC (none) -> C28323
- C2: renamed from C8; LCSC (none) -> C28233
- D1: renamed from D3; LCSC (none) -> C22452
- J1: LCSC (none) -> C5338271
- Motor1, Motor2: LCSC (none) -> C277598
- R1: renamed from R4; LCSC (none) -> C27834
- R2: renamed from R3; LCSC (none) -> C27834
- R_En1: renamed from R1; LCSC (none) -> C17408
- R_boot1: renamed from R2; LCSC (none) -> C17408
- U1: renamed from U3; LCSC (none) -> C354068
- U2: LCSC (none) -> C969102
- U3: renamed from U1; LCSC (none) -> C2913197
- mosfet1: renamed from Trans_1; footprint CONN_SD-502352-001_02_MOL -> Connector_4:CONN_SD-502352-001_02_MOL; LCSC (none) -> C114107
- mosfet2: renamed from Trans_2; footprint CONN_SD-502352-001_02_MOL -> Connector_4:CONN_SD-502352-001_02_MOL; LCSC (none) -> C114107
- mosfet3: renamed from Trans_3; footprint CONN_SD-502352-001_02_MOL -> Connector_4:CONN_SD-502352-001_02_MOL; LCSC (none) -> C114107
- mosfet4: renamed from mosfet1; LCSC (none) -> C9114
- mosfet5: renamed from mosfet2; LCSC (none) -> C9114
- mosfet6: renamed from mosfet3; LCSC (none) -> C9114
- motorc1: renamed from motor1_c1; value C_Polarized -> 100uF; footprint Capacitor_THT:CP_Radial_D6.3mm_P2.50mm -> Capacitor_SMD:CP_Elec_6.3x5.4; LCSC (none) -> C2749
- motorc2: renamed from motor2_c1; value C_Polarized -> 100uF; footprint Capacitor_THT:CP_Radial_D6.3mm_P2.50mm -> Capacitor_SMD:CP_Elec_6.3x5.4; LCSC (none) -> C2749
- power1: renamed from J4; LCSC (none) -> C5188434; now in the parts list
- smooth_cap1: renamed from esp_smoothingcaps_1; Label (none) -> C1711
- smooth_cap2: renamed from esp_smoothingcaps_2; Label (none) -> C1711
- tr1: renamed from tr3; LCSC (none) -> C17513
- tr2: LCSC (none) -> C17513
- tr3: renamed from tr1; LCSC (none) -> C17513
- vd1: renamed from VoltageDivider1; LCSC (none) -> C277598
- vd_c1: renamed from vd_c4; LCSC (none) -> C377773
- vd_c2: renamed from vd_c3; LCSC (none) -> C123143
- vd_r1: LCSC (none) -> C2933447
- renumbered J3 to IO1, J2 to input1
Other:
- moved on the sheet: 5Vout1
