File: V67_cycletron.kicad_sch (KiCad schematic)
At the start: 54 parts, among them J1 USB_C_Receptacle_USB2.0_16P, J3 Screw_Terminal_01x11, U1 LM1117DT-5.0, U2 LM1117DT-3.3, U4 ESP32-S3-WROOM-1

Commit message: edited silkscreen
Parts:
- removed D5: LED, LED_SMD:LED_0603_1608Metric_Pad1.05x0.95mm_HandSolder, symbol Device:LED
- removed R4: 4.7k, Resistor_SMD:R_0805_2012Metric_Pad1.20x1.40mm_HandSolder, symbol Device:R
