File: _autosave-V67_cycletron.kicad_pcb (KiCad board)
At the start: 4 copper layers, 102.1 x 110.1 mm, 55 parts, among them J1 USB_C_Receptacle_USB2.0_16P, J3 Screw_Terminal_01x11, U1 LM1117DT-5.0, U2 LM1117DT-3.3, U4 ESP32-S3-WROOM-1

Commit message: updates from laptop airport
Parts:
- moved mccap1 173.0 mm to (219.4, 35.9)
- moved C1 173.0 mm to (213.3, 36.0)
- moved C2 173.0 mm to (210.3, 36.0)
- moved mccap2 173.0 mm to (216.3, 36.0)
- moved Motor_1 170.2 mm to (245.1, 64.8)
- moved motorc1 167.1 mm to (268.0, 60.7), turned to 90 degrees
- moved motorc2 154.7 mm to (268.5, 44.0), turned to 90 degrees
- moved Motor_2 152.1 mm to (245.3, 48.5)
- moved Boot1 10.6 mm to (218.5, 43.5)
- moved R_boot1 10.6 mm to (218.5, 46.5)
- moved R_En1 5.52 mm to (213.0, 39.0), turned to 180 degrees
- moved En1 4.50 mm to (218.6, 40.0)
Routing:
- net BOOT: track 111.4 -> 95.5 mm
- net +12V: track 64.5 -> 76.3 mm
- net En: track 60.8 -> 49.5 mm
- net 3V3: track 74.9 -> 81.0 mm
- net GND: track 15.2 -> 15.3 mm, vias 37 -> 41
