File: V67_cycletron.kicad_pcb (KiCad board)
At the start: 4 copper layers, 102.1 x 110.1 mm, 55 parts, among them J1 USB_C_Receptacle_USB2.0_16P, J3 Screw_Terminal_01x11, U1 LM1117DT-5.0, U2 LM1117DT-3.3, U4 ESP32-S3-WROOM-1

Commit message: board layout redesign
Parts:
- removed ? (x4): , 
- removed D1, D2, D3: D_Schottky, Diode_SMD:D_SMA
- removed IO1, IO2, IO3, IO4, mosfet1, mosfet2, mosfet3: 5023520200, Connector_4:CONN_SD-502352-001_02_MOL
- removed mosfet4, mosfet5, mosfet6: HD2305, Package_TO_SOT_SMD:SOT-23
- removed power3, power5: Screw_Terminal_01x02, TerminalBlock:TerminalBlock_MaiXu_MX126-5.0-02P_1x02_P5.00mm
- removed tr1, tr2, tr3: 1k, Resistor_SMD:R_0805_2012Metric_Pad1.20x1.40mm_HandSolder
- moved R_En1 118.3 mm to (109.7, 85.0)
- moved En1 114.9 mm to (115.3, 86.0)
- moved J1 113.1 mm to (98.9, 76.5)
- moved U2 113.1 mm to (101.1, 90.8)
- moved 3v3in1 113.1 mm to (82.2, 98.5)
- moved 3v3out1 113.1 mm to (108.2, 89.5)
- moved 5Vin1 113.1 mm to (82.2, 91.0)
- moved 5Vout1 113.1 mm to (90.7, 78.8)
- moved D4 113.1 mm to (107.8, 94.0)
- moved Dpower1 113.1 mm to (81.2, 85.5)
- moved R1 113.1 mm to (96.2, 83.0)
- moved R2 113.1 mm to (101.2, 83.0)
- moved U1 113.1 mm to (92.2, 91.0)
- moved U4 113.1 mm to (128.2, 86.5)
- moved input1 113.1 mm to (81.6, 77.4)
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Routing:
- net BOOT: track 111.4 -> 22.9 mm, vias 4 -> 2
- net D+: track 108.3 -> 31.4 mm, vias 4 -> 2
- net D-: track 105.8 -> 30.2 mm, vias 4 -> 2
- net 3V3: track 74.9 -> 14.8 mm
- net IO4: track 59.8 -> 0.00 mm
- net Motor2_EN: track 55.3 -> 0.00 mm
- net I20: track 54.9 -> 0.00 mm
- net Motor2_M0: track 53.2 -> 0.00 mm
- net mosfet3_i: track 52.2 -> 0.00 mm
- net +5V: track 104.9 -> 52.7 mm, vias 3 -> 0
- net I19: track 49.8 -> 0.00 mm
- net +12V: track 64.5 -> 14.8 mm, vias 4 -> 0
- net Motor2_M1: track 48.9 -> 0.00 mm
- net IO5: track 48.4 -> 0.00 mm
- net Motor2_M2: track 46.4 -> 0.00 mm
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- removed copper zone on F.Cu, net +12V
- removed copper zone on F.Cu, net 3V3
- removed copper zone on B.Cu, net GND
Other:
- board size 102.1 x 110.1 mm -> 101.9 x 49.8 mm
- board text removed: "-"
- board text removed: "10"
- board text removed: "11"
- board text removed: "12"
- board text removed: "15"
- board text removed: "16"
- board text removed: "17"
- board text removed: "18"
- board text removed: "19"
- board text removed: "20"
- board text removed: "3v3"
- board text removed: "4"
- board text removed: "5"
- board text removed: "6"
- board text removed: "7"
- board text removed: "8"
- board text removed: "9"
- board text removed: "Dev: Ryan Taylor"
- board text removed: "ESP32-S3-WROOM-1-N16"
- board text removed: "GND"
- board text removed: "input"
